File: Tardygrade.kicad_pcb (KiCad board)
At the start: 2 copper layers, 50 x 50 mm, 23 parts, among them J1 Conn_01x03, J2 Conn_01x03, J3 Conn_01x03, J4 Conn_01x03, J5 Conn_01x03_Male, U1 MCP1642B, U2 HUZZAH32, U3 Tinypico, U4 HallSwitch, U5 HallSwitch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

Commit message: Version 0.42
Parts:
- added R2: 1k, Resistor_SMD:R_0603_1608Metric_Pad0.98x0.95mm_HandSolder, B.Cu at (105.8, 102.2)
- added R3: 2k, Resistor_SMD:R_0603_1608Metric_Pad0.98x0.95mm_HandSolder, B.Cu at (104.7, 103.4)
- added R4: 1k, Resistor_SMD:R_0603_1608Metric_Pad0.98x0.95mm_HandSolder, B.Cu at (103.2, 104.9)
- added R5: 2k, Resistor_SMD:R_0603_1608Metric_Pad0.98x0.95mm_HandSolder, B.Cu at (102.0, 106.0)
- C1, C2: footprint Capacitor_SMD:C_0603_1608Metric_Pad1.08x0.95mm_HandSolder -> 222footprints:C_0603_1608Metric_HandSolderBig
Connections:
- J3 pad 2: 3V3_Rail -> 5V_Rail
- J3 pad 3: LidarFront -> Net-(J3-Pad3)
- J4 pad 2: 3V3_Rail -> 5V_Rail
- J4 pad 3: LidarRear -> Net-(J4-Pad3)
- U1 pad 1: 3V3_Rail -> 5V_Rail
- U1 pad 2: Net-(U1-Pad2) -> unconnected-(U1-Pad2)
- U1 pad 3: Net-(U1-Pad3) -> unconnected-(U1-Pad3)
- U2 pad 24: Net-(U2-Pad24) -> GPIO12
- U2 pad 25: Net-(U2-Pad25) -> unconnected-(U2-Pad25)
- U2 pad 26: Net-(U2-Pad26) -> unconnected-(U2-Pad26)
- U2 pad 3: Net-(U2-Pad3) -> unconnected-(U2-Pad3)
- U3 pad 16: Net-(U3-Pad16) -> EN
- U3 pad 18: Net-(U3-Pad18) -> unconnected-(U3-Pad18)
- X1 pad 7: Net-(X1-Pad7) -> GPIO12
Routing:
- net Net-(J4-Pad3): track 0.00 -> 20.4 mm
- net LidarRear: track 30.3 -> 11.3 mm
- net EN: track 10.6 -> 29.2 mm, vias 0 -> 1
- net Net-(J3-Pad3): track 0.00 -> 17.9 mm
- net LidarFront: track 31.9 -> 16.0 mm
- net GPIO12: track 0.00 -> 14.3 mm, vias 0 -> 1
- net 3V3_Rail: track 111.4 -> 97.7 mm
- net 5V_Rail: track 111.0 -> 124.7 mm
- net Reset: track 86.5 -> 87.9 mm
- net HallRight: track 36.0 -> 36.8 mm
- net GND: vias 37 -> 40
Other:
- net class Default removed
- board text added: "Tardygrade"
- board text added: "v0.42"
- board text added: "© Dejan Ristic 2023"
- board text removed: "Tardygrade v0.41"
